Commit message: updated texture

File: gym_flexassembly/data/robots/barrett-bh8/model.urdf (robot description, URDF)
Before this commit: robot barrett-bh8, 14 links, 13 joints
Links:
- link bhand_palm_link: geometry collision box size=0.024 0.108 0.033; collision box size=0.076 0.046 0.012
- link finger_1/dist_link: geometry collision mesh filename=barrett-bh8/meshes/sw_meshes/bhand/bhand_finger_dist_link_c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; visual mesh filename=barrett-bh8/meshes/sw_meshes/bhand/dist_fine.obj
- link finger_1/med_link: geometry collision box size=0.031 0.023 0.019; collision box size=0.07 0.019 0.006
- link finger_1/prox_link: geometry collision box size=0.066 0.024 0.033; collision cylinder length=0.024 radius=0.015
- link finger_2/dist_link: geometry collision mesh filename=barrett-bh8/meshes/sw_meshes/bhand/bhand_finger_dist_link_c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; visual mesh filename=barrett-bh8/meshes/sw_meshes/bhand/dist_fine.obj
- link finger_2/med_link: geometry collision box size=0.031 0.023 0.019; collision box size=0.07 0.019 0.006
- link finger_2/prox_link: geometry collision box size=0.066 0.024 0.033; collision cylinder length=0.024 radius=0.015
- link finger_3/dist_link: geometry collision mesh filename=barrett-bh8/meshes/sw_meshes/bhand/bhand_finger_dist_link_c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; visual mesh filename=barrett-bh8/meshes/sw_meshes/bhand/dist_fine.obj
- link finger_3/med_link: geometry collision box size=0.031 0.023 0.019; collision box size=0.07 0.019 0.006
