Commit message: polishing update

File: gym_flexassembly/data/objects/window.urdf (robot description, URDF)
Before this commit: robot window, 2 links, 1 joints
Links:
- link frame_link: geometry collision mesh filename=WindowFrame.obj scale=1 0.7 0.6; visual mesh filename=WindowFrame.obj scale=1 0.7 0.6
- link window_link: geometry collision mesh filename=Window.obj scale=1 0.7 0.6; visual mesh filename=Window.obj scale=1 0.7 0.6
