Commit message: urdf update

File: gym_flexassembly/data/robots/epfl-iiwa14/iiwa14_mod.urdf (robot description, URDF)
Before this commit: robot iiwa14, 15 links, 14 joints
Links:
- removed link SchunkEGP40_Finger1_link
- removed link SchunkEGP40_Finger2_link
- link iiwa_link_ee: mass 0.6 -> 0.68
Joints:
- removed joint SchunkEGP40_Finger1_joint
- removed joint SchunkEGP40_Finger2_joint
- joint iiwa_joint_ee: origin xyz=0 0 0.001 rpy=0 0 0 -> xyz=0 0 0.115 rpy=0 0 0

Commit message: qp test

File: gym_flexassembly/data/robots/epfl-iiwa14/iiwa14_mod.urdf (robot description, URDF)
Before this commit: robot iiwa14, 13 links, 12 joints
Links:
- link iiwa_link_ee: mass 0.68 -> 0.822
Joints:
- joint iiwa_joint_ee: origin xyz=0.081 0 -0.0249 rpy=0 0 0 -> xyz=0.081 0 0.1351 rpy=0 0 0
