Commit message: Mount camera to robot arm

File: gym_flexassembly/data/robots/epfl-iiwa14/iiwa14.urdf (robot description, URDF)
Before this commit: robot iiwa14, 13 links, 12 joints
Links:
- added link camera_mount, mass 0.215; collision mesh filename=model://epfl-iiwa14/meshes/camera/camera_mount.obj; visual mesh filename=model://epfl-iiwa14/meshes/camera/camera_mount.obj
- added link realsense_camera, mass 0.215; collision mesh filename=model://epfl-iiwa14/meshes/camera/RealSense_D435.obj; visual mesh filename=model://epfl-iiwa14/meshes/camera/RealSense_D435.obj
- link iiwa_link_0: geometry collision mesh filename=model://epfl-iiwa14/meshes/iiwa14/collision/link_0.stl; visual mesh filename=model://epfl-iiwa14/meshes/iiwa14/visual/link_0.obj
- link iiwa_link_1: geometry collision mesh filename=model://epfl-iiwa14/meshes/iiwa14/collision/link_1.stl; visual mesh filename=model://epfl-iiwa14/meshes/iiwa14/visual/link_1.obj
- link iiwa_link_2: geometry collision mesh filename=model://epfl-iiwa14/meshes/iiwa14/collision/link_2.stl; visual mesh filename=model://epfl-iiwa14/meshes/iiwa14/visual/link_2.obj
- link iiwa_link_3: geometry collision mesh filename=model://epfl-iiwa14/meshes/iiwa14/collision/link_3.stl; visual mesh filename=model://epfl-iiwa14/meshes/iiwa14/visual/link_3.obj
- link iiwa_link_4: geometry collision mesh filename=model://epfl-iiwa14/meshes/iiwa14/collision/link_4.stl; visual mesh filename=model://epfl-iiwa14/meshes/iiwa14/visual/link_4.obj
- link iiwa_link_5: geometry collision mesh filename=model://epfl-iiwa14/meshes/iiwa14/collision/link_5.stl; visual mesh filename=model://epfl-iiwa14/meshes/iiwa14/visual/link_5.obj
- link iiwa_link_6: geometry collision mesh filename=model://epfl-iiwa14/meshes/iiwa14/collision/link_6.stl; visual mesh filename=model://epfl-iiwa14/meshes/iiwa14/visual/link_6.obj
- link iiwa_link_7: geometry collision mesh filename=model://epfl-iiwa14/meshes/iiwa14/collision/link_7.stl; visual mesh filename=model://epfl-iiwa14/meshes/iiwa14/visual/link_7.obj
Joints:
- added joint iiwa7_joint_camera_mount: type fixed, parent ft_sensor, child camera_mount, origin xyz=0 0 0.015 rpy=0 0 0
- added joint iiwa7_joint_camera_mount_realsense: type fixed, parent camera_mount, child realsense_camera, origin xyz=-0.081 0 0.0259 rpy=3.14159 0 1.5708
- joint iiwa7_joint_ee: origin xyz=0 0 0.01 rpy=0 0 0 -> xyz=0 0 0.001 rpy=0 0 0; parent ft_sensor -> camera_mount

Commit message: test urdf

File: gym_flexassembly/data/robots/epfl-iiwa14/iiwa14.urdf (robot description, URDF)
Before this commit: robot iiwa14, 15 links, 14 joints
Joints:
- joint iiwa_joint_ee: origin xyz=0 0 0.001 rpy=0 0 0 -> xyz=0.081 0 -0.0249 rpy=0 0 0; parent camera_mount -> realsense_camera

File: gym_flexassembly/data/robots/epfl-iiwa14/iiwa14_mod.urdf (robot description, URDF)
Before this commit: robot iiwa14, 13 links, 12 joints
Joints:
- joint iiwa_joint_ee: origin xyz=0 0 0.115 rpy=0 0 0 -> xyz=0.081 0 -0.0249 rpy=0 0 0; parent camera_mount -> realsense_camera

Commit message: update urdf to have no branch

File: gym_flexassembly/data/robots/epfl-iiwa14/iiwa14.urdf (robot description, URDF)
Before this commit: robot iiwa14, 15 links, 14 joints
Joints:
- joint iiwa_joint_camera_mount_realsense: origin xyz=-0.081 0 0.0259 rpy=3.14159 0 1.5708 -> xyz=-0.081 0 0.0259 rpy=0 0 0

File: gym_flexassembly/data/robots/epfl-iiwa14/iiwa14_mod.urdf (robot description, URDF)
Before this commit: robot iiwa14, 13 links, 12 joints
Joints:
- joint iiwa_joint_camera_mount_realsense: origin xyz=-0.081 0 0.0259 rpy=3.14159 0 1.5708 -> xyz=-0.081 0 0.0259 rpy=0 0 0

Commit message: fixed gripper collision objects

File: gym_flexassembly/data/robots/epfl-iiwa14/iiwa14.urdf (robot description, URDF)
Before this commit: robot iiwa14, 15 links, 14 joints
Links:
- link SchunkEGP40_Finger1_link: geometry collision box size=0.0195 0.03 0.04985; visual mesh filename=model://schunk-egp-40/meshes/visual/dae/schunk-egp-40-finge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 scale=1 1 1
- link SchunkEGP40_Finger2_link: geometry collision box size=0.0195 0.03 0.04985; visual mesh filename=model://schunk-egp-40/meshes/visual/dae/schunk-egp-40-finge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 scale=1 1 1

Commit message: updated urdf grasp frame

File: gym_flexassembly/data/robots/epfl-iiwa14/iiwa14.urdf (robot description, URDF)
Before this commit: robot iiwa14, 15 links, 14 joints
Joints:
- joint SchunkEGP40_Finger1_joint: origin xyz=0.006800 0.000500 0.108000 rpy=0 0 0 -> xyz=0.006800 0.000500 -0.02 rpy=0 0 0
- joint SchunkEGP40_Finger2_joint: origin xyz=-0.006800 0.000500 0.108000 rpy=0 0 3.14 -> xyz=-0.006800 0.000500 -0.02 rpy=0 0 3.14
- joint iiwa_joint_ee: origin xyz=0.081 0 -0.0249 rpy=0 0 0 -> xyz=0.081 0 0.1031 rpy=0 0 0

Commit message: save all

File: gym_flexassembly/data/robots/epfl-iiwa14/iiwa14.urdf (robot description, URDF)
Before this commit: robot iiwa14, 15 links, 14 joints
Joints:
- joint iiwa_joint_ee: origin xyz=0.081 0 0.1031 rpy=0 0 0 -> xyz=0.081 0 0.2 rpy=0 0 0

Commit message: updated robot model

File: gym_flexassembly/data/robots/epfl-iiwa14/iiwa14.urdf (robot description, URDF)
Before this commit: robot iiwa14, 15 links, 14 joints
Joints:
- joint SchunkEGP40_Finger1_joint: origin xyz=0.006800 0.000500 -0.02 rpy=0 0 0 -> xyz=0.006800 0.000500 -0.052 rpy=0 0 0
- joint SchunkEGP40_Finger2_joint: origin xyz=-0.006800 0.000500 -0.02 rpy=0 0 3.14 -> xyz=-0.006800 0.000500 -0.052 rpy=0 0 3.14
- joint iiwa_joint_ee: origin xyz=0.081 0 0.2 rpy=0 0 0 -> xyz=0.081 0 0.1351 rpy=0 0 0

Commit message: saved from robot

File: gym_flexassembly/data/robots/epfl-iiwa14/iiwa14.urdf (robot description, URDF)
Before this commit: robot iiwa14, 13 links, 12 joints
Links:
- link SchunkEGP40_Finger1_link: mass 0.04 -> 0.015
- link SchunkEGP40_Finger2_link: mass 0.04 -> 0.015
- link ft_sensor: mass 0.215 -> 0.283
- link iiwa7_link_ee: mass 0.6 -> 0.822

Commit message: update mass parameters

File: gym_flexassembly/data/robots/epfl-iiwa14/iiwa14.urdf (robot description, URDF)
Before this commit: robot iiwa14, 15 links, 14 joints
Links:
- link SchunkEGP40_Finger1_link: mass 0.04 -> 0.015
- link SchunkEGP40_Finger2_link: mass 0.04 -> 0.015
- link ft_sensor: mass 0.215 -> 0.283
- link iiwa_link_ee: mass 0.6 -> 0.822

Commit message: added stuff for sim mirroring

File: gym_flexassembly/data/robots/epfl-iiwa14/iiwa14.urdf (robot description, URDF)
Before this commit: robot iiwa14, 15 links, 14 joints
Joints:
- joint iiwa_joint_ft_sensor: origin xyz=0 0 0.059 rpy=0 0 0 -> xyz=0 0 0.059 rpy=0 0 -0.785398

Commit message: update

File: gym_flexassembly/data/robots/epfl-iiwa14/iiwa14.urdf (robot description, URDF)
Before this commit: robot iiwa14, 15 links, 14 joints
Joints:
- joint iiwa_joint_ee: origin xyz=0.081 0 0.1351 rpy=0 0 0 -> xyz=0.081 0 0.1621 rpy=0 0 0
- joint iiwa_joint_ft_sensor: origin xyz=0 0 0.059 rpy=0 0 -0.785398 -> xyz=0 0 0.059 rpy=0 0 0

File: gym_flexassembly/data/robots/epfl-iiwa14/iiwa14_mod.urdf (robot description, URDF)
Before this commit: robot iiwa14, 13 links, 12 joints
Joints:
- joint iiwa_joint_ee: origin xyz=0.081 0 0.1351 rpy=0 0 0 -> xyz=0.081 0 0.1621 rpy=0 0 0
- joint iiwa_joint_ft_sensor: origin xyz=0 0 0.059 rpy=0 0 -0.785398 -> xyz=0 0 0.059 rpy=0 0 0
