Commit message: update rail integration

File: gym_flexassembly/data/flexassembly/rail.urdf (robot description, URDF)
Before this commit: robot rail.urdf, 1 links, 0 joints
Links:
- link baseLink: geometry collision mesh filename=Rail_Coll.obj scale=1 1 1; visual mesh filename=Rail.obj scale=1 1 1

Commit message: clamp update

File: gym_flexassembly/data/flexassembly/rail.urdf (robot description, URDF)
Before this commit: robot rail.urdf, 1 links, 0 joints
Links:
- link baseLink: geometry collision mesh filename=Rail_Coll.obj scale=1 1.15 1; visual mesh filename=Rail.obj scale=1 1.15 1
